File: dongle/sch/wirelessness.sch (KiCad schematic (older format))
At the start: 16 parts, among them IC1 ATMEGA8A-P, J1 DB9, P1 NRF24L01, SW10 SW_PUSH, SW9 SW_PUSH, U1 NCP1117ST33T3G, X1 12M

Commit message: controller implementation of all buttons, clean-up
Parts:
- removed C3: 10u, symbol CAPAPOL
Connections:
- no-connect marks 11 -> 12
Other:
- note added: "The buttons and the LED are left for debugging purposes only."
- note removed: "The buttons and the LED are left for debugging purpose only."
- moved on the sheet: C4
Changed lines of the file:
@@
 L C C4
 U 1 1 59C88AFC
-P 9100 5850
-F 0 "C4" H 9100 5950 40  0000 L CNN
-F 1 "100n" H 9106 5765 40  0000 L CNN
-F 2 "" H 9138 5700 30  0000 C CNN
-F 3 "" H 9100 5850 60  0000 C CNN
-	1    9100 5850
-	1    0    0    -1
-$EndComp
-$Comp
-L CAPAPOL C3
-U 1 1 59C88B57
-P 8600 5850
-F 0 "C3" H 8650 5950 40  0000 L CNN
-F 1 "10u" H 8650 5750 40  0000 L CNN
-F 2 "" H 8700 5700 30  0000 C CNN
-F 3 "" H 8600 5850 300 0000 C CNN
-	1    8600 5850
+P 9050 5850
+F 0 "C4" H 9050 5950 40  0000 L CNN
+F 1 "100n" H 9056 5765 40  0000 L CNN
+F 2 "" H 9088 5700 30  0000 C CNN
+F 3 "" H 9050 5850 60  0000 C CNN
+	1    9050 5850
 	1    0    0    -1
 $EndComp
@@
 L GND #PWR014
 U 1 1 59C88BB0
-P 8850 6150
-F 0 "#PWR014" H 8850 6150 30  0001 C CNN
-F 1 "GND" H 8850 6080 30  0001 C CNN
-F 2 "" H 8850 6150 60  0001 C CNN
-F 3 "" H 8850 6150 60  0001 C CNN
-	1    8850 6150
+P 9050 6150
+F 0 "#PWR014" H 9050 6150 30  0001 C CNN
+F 1 "GND" H 9050 6080 30  0001 C CNN
+F 2 "" H 9050 6150 60  0001 C CNN
+F 3 "" H 9050 6150 60  0001 C CNN
+	1    9050 6150
 	1    0    0    -1
 $EndComp
@@
 L 3V3 #PWR015
 U 1 1 59C88D24
-P 8850 5550
-F 0 "#PWR015" H 8850 5650 40  0001 C CNN
-F 1 "3V3" H 8850 5675 40  0000 C CNN
-F 2 "" H 8850 5550 60  0001 C CNN
-F 3 "" H 8850 5550 60  0001 C CNN
-	1    8850 5550
+P 9050 5550
+F 0 "#PWR015" H 9050 5650 40  0001 C CNN
+F 1 "3V3" H 9050 5675 40  0000 C CNN
+F 2 "" H 9050 5550 60  0001 C CNN
+F 3 "" H 9050 5550 60  0001 C CNN
+	1    9050 5550
 	1    0    0    -1
 $EndComp
-Wire Wire Line
-	8600 5650 8600 5600
-Wire Wire Line
-	8600 5600 9100 5600
-Wire Wire Line
-	9100 5600 9100 5650
-Wire Wire Line
-	8850 5550 8850 5600
-Connection ~ 8850 5600
-Wire Wire Line
-	8600 6050 8600 6100
-Wire Wire Line
-	8600 6100 9100 6100
-Wire Wire Line
-	9100 6100 9100 6050
-Wire Wire Line
-	8850 6150 8850 6100
-Connection ~ 8850 6100
 $Comp
 L PWR_FLAG #FLG016
@@
 NoConn ~ 6500 2800
 Text Notes 3750 7400 0    60   ~ 0
-The buttons and the LED are left for debugging purpose only.
+The buttons and the LED are left for debugging purposes only.
 $Comp
 L R R1
@@
 	9500 3750 9500 3800
 Connection ~ 9500 3800
+NoConn ~ 10200 3200
+Wire Wire Line
+	9050 6050 9050 6150
+Wire Wire Line
+	9050 5550 9050 5650
 $EndSCHEMATC
